Commit message: araçların yapısını değiştirdim

File: src/robots/robot_designs/lidar.xacro (robot description, xacro)
@@ -23,5 +23,5 @@
         <parent link="base_link"/>
         <child link="lidar_link"/>
-        <origin xyz="0 0 0.075" rpy="0 0 0"/>
+        <origin xyz="0.1 0 0.15" rpy="0 0 0"/>
     </joint>
     <gazebo reference="lidar_link">

File: src/robots/robot_designs/turtlebot_core.xacro (robot description, xacro)
@@ -1,12 +1,13 @@
 <?xml version="1.0"?>
 <robot xmlns:xacro="http://www.ros.org/wiki/xacro">
-    <xacro:property name="base_radius" value="0.15"/>
-    <xacro:property name="base_length" value="0.1"/>
+    <xacro:property name="box_length" value="0.5"/>
+    <xacro:property name="box_width" value="0.4"/>
+    <xacro:property name="box_height" value="0.2"/>
     <xacro:property name="wheel_radius" value="0.05"/>
-    <xacro:property name="wheel_thickness" value="0.02"/>
+    <xacro:property name="wheel_thickness" value="0.05"/>
     <link name="base_link">
         <visual>
             <geometry>
-                <cylinder radius="${base_radius}" length="${base_length}"/>
+                <box size="${box_length} ${box_width} ${box_height}"/>
             </geometry>
             <material name="blue">
@@ -16,5 +17,5 @@
         <collision>
             <geometry>
-                <cylinder radius="${base_radius}" length="${base_length}"/>
+                <box size="${box_length} ${box_width} ${box_height}"/>
             </geometry>
         </collision>
@@ -46,5 +47,5 @@
         <parent link="base_link"/>
         <child link="left_wheel"/>
-        <origin xyz="0 0.17 -0.05" rpy="-1.5708 0 0"/>
+        <origin xyz="-0.12 0.20 -0.1" rpy="-1.5708 0 0"/>
         <axis xyz="0 0 1"/>
     </joint>
@@ -69,5 +70,5 @@
         <parent link="base_link"/>
         <child link="right_wheel"/>
-        <origin xyz="0 -0.17 -0.05" rpy="-1.5708 0 0"/>
+        <origin xyz="-0.12 -0.20 -0.1" rpy="-1.5708 0 0"/>
         <axis xyz="0 0 1"/>
     </joint>
@@ -87,6 +88,6 @@
         </collision>
         <inertial>
-            <mass value="0.1"/>
-            <inertia ixx="0.0001" ixy="0" ixz="0" iyy="0.0001" iyz="0" izz="0.0001"/>
+            <mass value="0.05"/>
+            <inertia ixx="0.00001" ixy="0" ixz="0" iyy="0.00001" iyz="0" izz="0.00001"/>
         </inertial>
     </link>
@@ -94,5 +95,10 @@
         <parent link="base_link"/>
         <child link="caster_wheel"/>
-        <origin xyz="0.1 0 -0.05" rpy="0 0 0"/>
+        <origin xyz="0.15 0 -0.1" rpy="0 0 0"/>
     </joint>
+    <gazebo reference="caster_wheel">
+        <mu1>0.0</mu1>
+        <mu2>0.0</mu2>
+        <material>Gazebo/White</material>
+    </gazebo>
 </robot>
