Commit message: Multi robot güncellemesi

File: src/robots/robot_designs/lidar.xacro (robot description, xacro)
@@ -1,5 +1,5 @@
 <?xml version="1.0"?>
 <robot xmlns:xacro="http://www.ros.org/wiki/xacro">
-    <link name="lidar_link">
+    <link name="${prefix}lidar_link">
         <visual>
             <geometry>
@@ -20,10 +20,10 @@
         </inertial>
     </link>
-    <joint name="lidar_joint" type="fixed">
-        <parent link="base_link"/>
-        <child link="lidar_link"/>
+    <joint name="${prefix}lidar_joint" type="fixed">
+        <parent link="${prefix}base_link"/>
+        <child link="${prefix}lidar_link"/>
         <origin xyz="0.1 0 0.15" rpy="0 0 0"/>
     </joint>
-    <gazebo reference="lidar_link">
+    <gazebo reference="${prefix}lidar_link">
         <sensor name="lidar_sensor" type="ray">
             <pose>0 0 0 0 0 0</pose>
@@ -50,5 +50,5 @@
                 </ros>
                 <output_type>sensor_msgs/LaserScan</output_type>
-                <frame_name>lidar_link</frame_name>
+                <frame_name>${prefix}lidar_link</frame_name>
             </plugin>
         </sensor>

File: src/robots/robot_designs/turtlebot.urdf.xacro (robot description, xacro)
@@ -1,10 +1,12 @@
 <?xml version="1.0"?>
 <robot xmlns:xacro="http://www.ros.org/wiki/xacro" name="turtlebot">
+    <xacro:arg name="prefix" default=""/>
+    <xacro:property name="prefix" value="$(arg prefix)"/>
     <xacro:include filename="turtlebot_core.xacro" />
     <xacro:include filename="lidar.xacro" />
     <gazebo>
         <plugin name="diff_drive" filename="libgazebo_ros_diff_drive.so">
-            <left_joint>left_wheel_joint</left_joint>
-            <right_joint>right_wheel_joint</right_joint>
+            <left_joint>$(arg prefix)left_wheel_joint</left_joint>
+            <right_joint>$(arg prefix)right_wheel_joint</right_joint>
             <wheel_separation>0.34</wheel_separation>
             <wheel_diameter>0.10</wheel_diameter>
@@ -15,6 +17,6 @@
             <publish_odom_tf>true</publish_odom_tf>
             <publish_wheel_tf>true</publish_wheel_tf>
-            <odometry_frame>odom</odometry_frame>
-            <robot_base_frame>base_link</robot_base_frame>
+            <odometry_frame>$(arg prefix)odom</odometry_frame>
+            <robot_base_frame>$(arg prefix)base_link</robot_base_frame>
         </plugin>
     </gazebo>

File: src/robots/robot_designs/turtlebot_core.xacro (robot description, xacro)
@@ -6,5 +6,5 @@
     <xacro:property name="wheel_radius" value="0.05"/>
     <xacro:property name="wheel_thickness" value="0.05"/>
-    <link name="base_link">
+    <link name="${prefix}base_link">
         <visual>
             <geometry>
@@ -25,5 +25,5 @@
         </inertial>
     </link>
-    <link name="left_wheel">
+    <link name="${prefix}left_wheel">
         <visual>
             <geometry>
@@ -44,11 +44,11 @@
         </inertial>
     </link>
-    <joint name="left_wheel_joint" type="continuous">
-        <parent link="base_link"/>
-        <child link="left_wheel"/>
+    <joint name="${prefix}left_wheel_joint" type="continuous">
+        <parent link="${prefix}base_link"/>
+        <child link="${prefix}left_wheel"/>
         <origin xyz="-0.12 0.20 -0.1" rpy="-1.5708 0 0"/>
         <axis xyz="0 0 1"/>
     </joint>
-    <link name="right_wheel">
+    <link name="${prefix}right_wheel">
         <visual>
             <geometry>
@@ -67,11 +67,11 @@
         </inertial>
     </link>
-    <joint name="right_wheel_joint" type="continuous">
-        <parent link="base_link"/>
-        <child link="right_wheel"/>
+    <joint name="${prefix}right_wheel_joint" type="continuous">
+        <parent link="${prefix}base_link"/>
+        <child link="${prefix}right_wheel"/>
         <origin xyz="-0.12 -0.20 -0.1" rpy="-1.5708 0 0"/>
         <axis xyz="0 0 1"/>
     </joint>
-    <link name="caster_wheel">
+    <link name="${prefix}caster_wheel">
         <visual>
             <geometry>
@@ -92,10 +92,10 @@
         </inertial>
     </link>
-    <joint name="caster_joint" type="fixed">
-        <parent link="base_link"/>
-        <child link="caster_wheel"/>
+    <joint name="${prefix}caster_joint" type="fixed">
+        <parent link="${prefix}base_link"/>
+        <child link="${prefix}caster_wheel"/>
         <origin xyz="0.15 0 -0.1" rpy="0 0 0"/>
     </joint>
-    <gazebo reference="caster_wheel">
+    <gazebo reference="${prefix}caster_wheel">
         <mu1>0.0</mu1>
         <mu2>0.0</mu2>
